Commit message: added ros2_control

File: humibot_description/urdf/robot.urdf.xacro (robot description, xacro)
@@ -5,5 +5,6 @@
    <xacro:include filename="utils/properties.xacro"/>
    <xacro:include filename="robot_core.xacro"/>
-   <xacro:include filename="gazebo_control.xacro"/>
+   <!-- <xacro:include filename="gazebo_control.xacro"/> -->
+   <xacro:include filename="ros2_control.xacro"/>
    <xacro:include filename="sensors/lidar.xacro"/>
 </robot>

File: humibot_description/urdf/sensors/lidar.xacro (robot description, xacro)
@@ -2,5 +2,5 @@
 <robot xmlns:xacro="http://www.ros.org/wiki/xacro">
    <joint name="lidar_joint" type="fixed">
-      <origin xyz="0.0 0.0 ${base_height+0.215}" rpy="0.0 0.0 0.0"/>
+      <origin xyz="0.0 0.0 ${base_height+0.215-0.0105}" rpy="0.0 0.0 0.0"/>
       <parent link="base_link"/>
       <child link="lidar_link"/>
@@ -8,5 +8,5 @@
    <link name="lidar_link">
       <visual>
-         <origin xyz="-0.053 -0.031 -0.0625" rpy="${pi/2} 0.0 ${pi/2}"/>
+         <origin xyz="-0.057 -0.031 -0.052" rpy="${pi/2} 0.0 ${pi/2}"/>
          <geometry>
                <mesh filename="package://humibot_description/meshes/ld06.stl" scale="0.001 0.001 0.001"/>
@@ -14,7 +14,7 @@
       </visual>
       <collision>
-         <origin xyz="0.005 0.0 -${0.05/2}" rpy="0.0 0.0 0.0"/>
+         <origin xyz="0 0 0" rpy="0 0 0"/>
          <geometry>
-            <box size="0.07 0.0672 0.05"/>
+            <cylinder radius="0.0175" length="0.015"/>
          </geometry>
       </collision>

Commit message: added ros2_control

File: humibot_description/urdf/robot.urdf.xacro (robot description, xacro)
@@ -1,10 +1,16 @@
 <?xml version="1.0" encoding="UTF-8"?>
 <robot xmlns:xacro="http://www.ros.org/wiki/xacro" name="humibot">
+   <xacro:arg name="use_ros2_control" default="True"/>
    <xacro:include filename="utils/colors.xacro"/>
    <xacro:include filename="utils/inertial_macros.xacro"/>
    <xacro:include filename="utils/properties.xacro"/>
    <xacro:include filename="robot_core.xacro"/>
-   <!-- <xacro:include filename="gazebo_control.xacro"/> -->
-   <xacro:include filename="ros2_control.xacro"/>
+   <!-- <xacro:include filename="ros2_control.xacro"/> -->
    <xacro:include filename="sensors/lidar.xacro"/>
+   <xacro:if value="$(arg use_ros2_control)">
+      <xacro:include filename="ros2_control.xacro"/>
+   </xacro:if>
+   <xacro:unless value="$(arg use_ros2_control)">
+      <xacro:include filename="gazebo_control.xacro"/>
+   </xacro:unless>
 </robot>

File: humibot_description/urdf/robot_core.xacro (robot description, xacro)
@@ -51,9 +51,7 @@
       </collision>
       <xacro:inertial_box mass="1.012" x="${base_length + 0.04}" y="${base_width}" z="${base_height+0.165}">
-         <origin xyz="${(base_length+0.0365)/2} 0.0 ${(base_height+0.165)/2}" rpy="0.0 0.0 0.0"/>
+         <origin xyz="${base_link_xoff + 0.037} 0.0 ${base_height/2}" rpy="0.0 0.0 0.0"/>
       </xacro:inertial_box>
    </link>
-   <!-- Dehumidifier -->
-   <!-- <xacro:include filename="sensors/dehumidifier.xacro"/> -->
    <!-- LEFT WHEEL -->
    <joint name="left_wheel_joint" type="continuous">
@@ -72,5 +70,5 @@
       <collision>
          <geometry>
-            <cylinder radius="${wheel_radius}" length="${wheel_width}"/>
+            <sphere radius="${wheel_radius}"/>
          </geometry>
       </collision>
@@ -95,5 +93,5 @@
       <collision>
          <geometry>
-            <cylinder radius="${wheel_radius}" length="${wheel_width}"/>
+            <sphere radius="${wheel_radius}"/>
          </geometry>
       </collision>
@@ -103,5 +101,5 @@
    </link>
    <!-- CASTER WHEEL -->
-   <joint name="caster_joint" type="fixed">
+   <joint name="front_caster_joint" type="fixed">
       <parent link="chassis_link"/>
       <child link="front_caster"/>
@@ -109,4 +107,31 @@
    </joint>
    <link name="front_caster">
+      <visual>
+         <geometry>
+            <sphere radius="${caster_radius}"/>
+         </geometry>
+         <material name="black"/>
+      </visual>
+      <collision>
+         <geometry>
+            <sphere radius="${caster_radius}"/>
+         </geometry>
+      </collision>
+      <visual name="caster_wheel_holder_visual">
+         <origin xyz="0.0 0.0 ${0.04/2}" rpy="0.0 0.0 0.0"/>
+         <geometry>
+            <box size="0.015 0.015 0.04"/>
+         </geometry>
+      </visual>
+      <xacro:inertial_sphere mass="${caster_mass}" radius="${caster_radius}">
+         <origin xyz="0 0 0" rpy="0 0 0"/>
+      </xacro:inertial_sphere>
+   </link>
+   <joint name="back_caster_joint" type="fixed">
+      <parent link="chassis_link"/>
+      <child link="back_caster"/>
+      <origin xyz="${(0.015/2) + 0.01} 0 ${-0.0125 - 0.005 + caster_radius - wheel_radius}" rpy="0 0 0"/>
+   </joint>
+   <link name="back_caster">
       <visual>
          <geometry>
@@ -145,3 +170,8 @@
       <mu2 value="0.001"/>
    </gazebo>
+   <gazebo reference="back_caster">
+      <material>Gazebo/Black</material>
+      <mu1 value="0.001"/>
+      <mu2 value="0.001"/>
+   </gazebo>
 </robot>

File: humibot_description/urdf/ros2_control.xacro (robot description, xacro)
@@ -1,5 +1,5 @@
 <?xml version="1.0" encoding="UTF-8"?>
 <robot xmlns:xacro="http://www.ros.org/wiki/xacro">
-   <ros2_control name="GazeboSystem" type="system">
+   <ros2_control name="RealSystem" type="system">
       <hardware>
          <plugin>gazebo_ros2_control/GazeboSystem</plugin>
@@ -22,4 +22,25 @@
       </joint>
    </ros2_control>
+   <!-- <ros2_control name="GazeboSystem" type="system">
+      <hardware>
+         <plugin>gazebo_ros2_control/GazeboSystem</plugin>
+      </hardware>
+      <joint name="left_wheel_joint">
+         <command_interface name="velocity">
+            <param name="min">-10</param>
+            <param name="max">10</param>
+         </command_interface>
+         <state_interface name="velocity"/>
+         <state_interface name="position"/>
+      </joint>
+      <joint name="right_wheel_joint">
+         <command_interface name="velocity">
+            <param name="min">-10</param>
+            <param name="max">10</param>
+         </command_interface>
+         <state_interface name="velocity"/>
+         <state_interface name="position"/>
+      </joint>
+   </ros2_control> -->
    <gazebo>
       <plugin name="gazebo_ros2_control" filename="libgazebo_ros2_control.so">

Commit message: fixed ros2_control gazebo

File: humibot_description/urdf/robot.urdf.xacro (robot description, xacro)
@@ -2,4 +2,5 @@
 <robot xmlns:xacro="http://www.ros.org/wiki/xacro" name="humibot">
    <xacro:arg name="use_ros2_control" default="True"/>
+   <xacro:arg name="use_sim_mode" default="False"/>
    <xacro:include filename="utils/colors.xacro"/>
    <xacro:include filename="utils/inertial_macros.xacro"/>

File: humibot_description/urdf/ros2_control.xacro (robot description, xacro)
@@ -1,56 +1,61 @@
 <?xml version="1.0" encoding="UTF-8"?>
 <robot xmlns:xacro="http://www.ros.org/wiki/xacro">
-   <ros2_control name="DiffDriveSystem" type="system">
-      <hardware>
-         <plugin>diffdrive_arduino/DiffDriveArduinoHardware</plugin>
-         <param name="left_wheel_name">left_wheel_joint</param>
-         <param name="right_wheel_name">right_wheel_joint</param>
-         <param name="loop_rate">30</param>
-         <param name="device">/dev/MotorController</param>
-         <param name="baud_rate">57600</param>
-         <param name="timeout_ms">1000</param>
-         <param name="enc_counts_per_rev">408</param>
-      </hardware>
-      <joint name="left_wheel_joint">
-         <command_interface name="velocity">
-            <param name="min">-10</param>
-            <param name="max">10</param>
-         </command_interface>
-         <state_interface name="position"/>
-         <state_interface name="velocity"/>
-      </joint>
-      <joint name="right_wheel_joint">
-         <command_interface name="velocity">
-            <param name="min">-10</param>
-            <param name="max">10</param>
-         </command_interface>
-         <state_interface name="position"/>
-         <state_interface name="velocity"/>
-      </joint>
-   </ros2_control>
-   <!-- <ros2_control name="GazeboSystem" type="system">
-      <hardware>
-         <plugin>gazebo_ros2_control/GazeboSystem</plugin>
-      </hardware>
-      <joint name="left_wheel_joint">
-         <command_interface name="velocity">
-            <param name="min">-10</param>
-            <param name="max">10</param>
-         </command_interface>
-         <state_interface name="velocity"/>
-         <state_interface name="position"/>
-      </joint>
-      <joint name="right_wheel_joint">
-         <command_interface name="velocity">
-            <param name="min">-10</param>
-            <param name="max">10</param>
-         </command_interface>
-         <state_interface name="velocity"/>
-         <state_interface name="position"/>
-      </joint>
-   </ros2_control> -->
+   <xacro:unless value="$(arg use_sim_mode)">
+      <ros2_control name="DiffDriveSystem" type="system">
+         <hardware>
+            <plugin>diffdrive_arduino/DiffDriveArduinoHardware</plugin>
+            <param name="left_wheel_name">left_wheel_joint</param>
+            <param name="right_wheel_name">right_wheel_joint</param>
+            <param name="loop_rate">30</param>
+            <param name="device">/dev/MotorController</param>
+            <param name="baud_rate">57600</param>
+            <param name="timeout_ms">1000</param>
+            <param name="enc_counts_per_rev">408</param>
+         </hardware>
+         <joint name="left_wheel_joint">
+            <command_interface name="velocity">
+               <param name="min">-10</param>
+               <param name="max">10</param>
+            </command_interface>
+            <state_interface name="position"/>
+            <state_interface name="velocity"/>
+         </joint>
+         <joint name="right_wheel_joint">
+            <command_interface name="velocity">
+               <param name="min">-10</param>
+               <param name="max">10</param>
+            </command_interface>
+            <state_interface name="position"/>
+            <state_interface name="velocity"/>
+         </joint>
+      </ros2_control>
+   </xacro:unless>
+   <xacro:if value="$(arg use_sim_mode)">
+      <ros2_control name="GazeboSystem" type="system">
+         <hardware>
+            <plugin>gazebo_ros2_control/GazeboSystem</plugin>
+         </hardware>
+         <joint name="left_wheel_joint">
+            <command_interface name="velocity">
+               <param name="min">-10</param>
+               <param name="max">10</param>
+            </command_interface>
+            <state_interface name="velocity"/>
+            <state_interface name="position"/>
+         </joint>
+         <joint name="right_wheel_joint">
+            <command_interface name="velocity">
+               <param name="min">-10</param>
+               <param name="max">10</param>
+            </command_interface>
+            <state_interface name="velocity"/>
+            <state_interface name="position"/>
+         </joint>
+      </ros2_control>
+   </xacro:if>
    <gazebo>
       <plugin name="gazebo_ros2_control" filename="libgazebo_ros2_control.so">
          <parameters>$(find humibot_bringup)/config/controllers.yaml</parameters>
+         <parameters>$(find humibot_bringup)/config/ros2_ctrl_use_sim.yaml</parameters>
       </plugin>
    </gazebo>
