Commit message: added slam_toolbox

File: humibot_description/urdf/gazebo_control.xacro (robot description, xacro)
@@ -13,5 +13,5 @@
          <!-- Output -->
          <odometry_frame>odom</odometry_frame>
-         <robot_base_frame>base_link</robot_base_frame>
+         <robot_base_frame>base_footprint</robot_base_frame>
          <publish_odom>true</publish_odom>
          <publish_odom_tf>true</publish_odom_tf>

File: humibot_description/urdf/robot_core.xacro (robot description, xacro)
@@ -1,5 +1,14 @@
 <?xml version="1.0" encoding="UTF-8"?>
 <robot xmlns:xacro="http://www.ros.org/wiki/xacro">
+   <!-- BASE FOOTPRINT -->
+   <link name="base_footprint">
+   </link>
    <!-- BASE LINK -->
+   <joint name="base_joint" type="fixed">
+      <!-- -${0.0125 + 0.005} -->
+      <origin xyz="0 0 ${wheel_zoff + wheel_radius}" rpy="0 0 0"/>
+      <parent link="base_link"/>
+      <child link="base_footprint"/>
+   </joint>
    <link name="base_link">
    </link>
@@ -50,5 +59,5 @@
          </geometry>
       </collision>
-      <xacro:inertial_box mass="1.012" x="${base_length + 0.04}" y="${base_width}" z="${base_height+0.165}">
+      <xacro:inertial_box mass="${base_mass}" x="${base_length + 0.04}" y="${base_width}" z="${base_height+0.165}">
          <origin xyz="${base_link_xoff + 0.037} 0.0 ${base_height/2}" rpy="0.0 0.0 0.0"/>
       </xacro:inertial_box>

File: humibot_description/urdf/sensors/lidar.xacro (robot description, xacro)
@@ -19,4 +19,7 @@
          </geometry>
       </collision>
+      <xacro:inertial_cylinder mass="0.109" length="0.015" radius="0.0175">
+         <origin xyz="0 0 0" rpy="0 0 0"/>
+      </xacro:inertial_cylinder>
    </link>
    <gazebo reference="lidar_link">

File: humibot_description/urdf/utils/properties.xacro (robot description, xacro)
@@ -10,16 +10,18 @@
    <xacro:property name="base_length" value="0.288"/>
    <xacro:property name="base_height" value="0.005"/>
-   <xacro:property name="base_mass" value="1.012"/>
+   <xacro:property name="base_mass" value="1.862"/>
    <xacro:property name="base_link_xoff" value="0.095"/>
    <xacro:property name="wheel_diameter" value="0.065"/>
    <xacro:property name="wheel_radius" value="${wheel_diameter/2}"/>
    <xacro:property name="wheel_width" value="0.026"/>
-   <xacro:property name="wheel_mass" value="0.057"/>
+   <xacro:property name="wheel_mass" value="0.048"/>
+   <xacro:property name="dc_motor_radius" value="0.0125"/>
+   <xacro:property name="dc_motor_length" value="0.063"/>
    <xacro:property name="wheel_ygap" value="0.01"/>
-   <xacro:property name="wheel_zoff" value="0.05"/>
+   <xacro:property name="wheel_zoff" value="${dc_motor_radius + 0.005}"/>
    <xacro:property name="wheel_xoff" value="0.12"/>
    <xacro:property name="caster_diameter" value="0.025"/>
    <xacro:property name="caster_radius" value="${caster_diameter/2}"/>
    <xacro:property name="caster_xoff" value="0.14"/>
-   <xacro:property name="caster_mass" value="0.017"/>
+   <xacro:property name="caster_mass" value="0.048"/>
 </robot>
